File: PCB/Starbie.kicad_pcb (KiCad board)
At the start: 2 copper layers, 120 x 99 mm, 7 parts, among them J1 Conn_01x04_Pin, J2 Conn_01x08_Pin, SW1 SW_Push, SW2 SW_Push, U1 XIAO-ESP32-C3-SMD, U2 DHT11

Commit message: added gerber files
Other:
- board text added: "Starbie"
